Commit message: fixing_bugs: #1

File: description/gazebo_controls.xacro (robot description, xacro)
@@ -9,6 +9,6 @@
             <right_joint>r_r_wheel_joint</right_joint>
             <!-- Wheel geometry -->
-            <wheel_separation>0.65</wheel_separation>
-            <wheel_radius>0.075</wheel_radius>
+            <wheel_separation>0.874</wheel_separation>
+            <wheel_radius>0.225</wheel_radius>
             <!-- Output -->
             <odom_publish_frequency>50</odom_publish_frequency>
@@ -19,4 +19,7 @@
             <child_frame_id>base_link</child_frame_id>
         </plugin>
+        <plugin filename="libignition-gazebo-joint-state-publisher-system.so" name="ignition::gazebo::systems::JointStatePublisher">
+            <topic>joint_states</topic>
+        </plugin>
     </gazebo>
 </robot>

File: description/joints.xacro (robot description, xacro)
@@ -14,5 +14,5 @@
         <parent link="base_link"/>
         <child link="l_r_wheel_link"/>
-        <axis xyz="0.0 -1.0 0.0"/>
+        <axis xyz="0.0 1.0 0.0"/>
     </joint>
     <joint name="r_r_wheel_joint" type="continuous">
@@ -20,5 +20,5 @@
         <parent link="base_link"/>
         <child link="r_r_wheel_link"/>
-        <axis xyz="0.0 -1.0 0.0"/>
+        <axis xyz="0.0 1.0 0.0"/>
     </joint>
     <joint name="r_f_wheel_joint" type="continuous">

File: description/links.xacro (robot description, xacro)
@@ -18,7 +18,7 @@
         </visual>
         <collision>
-            <origin xyz="0 0 0" rpy="0 0 1.5708"/>
-            <geometry>
-                <mesh filename="package://ros2-gz-vslam-bot/description/meshes/base_link.stl" scale="0.001 0.001 0.001"/>
+            <origin xyz="0.000973 0.000007 0.486096" rpy="0 0 0"/>
+            <geometry>
+                <box size="1.35 0.75 0.30"/>
             </geometry>
         </collision>
@@ -41,7 +41,7 @@
         </visual>
         <collision>
-            <origin xyz="-0.45 -0.325 -0.225" rpy="0 0 1.5708"/>
-            <geometry>
-                <mesh filename="package://ros2-gz-vslam-bot/description/meshes/left_front_wheel_link.stl" scale="0.001 0.001 0.001"/>
+            <origin xyz="0 0.11207 0" rpy="1.5708 0 0"/>
+            <geometry>
+                <cylinder radius="0.225" length="0.125"/>
             </geometry>
         </collision>
@@ -64,7 +64,7 @@
         </visual>
         <collision>
-            <origin xyz="-0.45 0.325 -0.225" rpy="0 0 1.5708"/>
-            <geometry>
-                <mesh filename="package://ros2-gz-vslam-bot/description/meshes/right_front_wheel_link.stl" scale="0.001 0.001 0.001"/>
+            <origin xyz="0 -0.11207 0" rpy="1.5708 0 0"/>
+            <geometry>
+                <cylinder radius="0.225" length="0.125"/>
             </geometry>
         </collision>
@@ -87,7 +87,7 @@
         </visual>
         <collision>
-            <origin xyz="0.45 -0.325 -0.225" rpy="0 0 1.5708"/>
-            <geometry>
-                <mesh filename="package://ros2-gz-vslam-bot/description/meshes/left_rear_wheel_link.stl" scale="0.001 0.001 0.001"/>
+            <origin xyz="0 0.11207 0" rpy="1.5708 0 0"/>
+            <geometry>
+                <cylinder radius="0.225" length="0.125"/>
             </geometry>
         </collision>
@@ -110,7 +110,7 @@
         </visual>
         <collision>
-            <origin xyz="0.45 0.325 -0.225" rpy="0 0 1.5708"/>
-            <geometry>
-                <mesh filename="package://ros2-gz-vslam-bot/description/meshes/right_rear_wheel_link.stl" scale="0.001 0.001 0.001"/>
+            <origin xyz="0 -0.11207 0" rpy="1.5708 0 0"/>
+            <geometry>
+                <cylinder radius="0.225" length="0.125"/>
             </geometry>
         </collision>
@@ -133,7 +133,7 @@
         </visual>
         <collision>
-            <origin xyz="-0.7 -0.225 -0.45" rpy="0 0 1.5708"/>
-            <geometry>
-                <mesh filename="package://ros2-gz-vslam-bot/description/meshes/front_bumper_link.stl" scale="0.001 0.001 0.001"/>
+            <origin xyz="0.071440 -0.225000 -0.018717" rpy="0 0 0"/>
+            <geometry>
+                <box size="0.12 0.95 0.5"/>
             </geometry>
         </collision>
@@ -156,8 +156,8 @@
         </visual>
         <collision>
-            <origin xyz="-0.6525 0 -0.705" rpy="0 0 1.5708"/>
-            <geometry>
-            <mesh filename="package://ros2-gz-vslam-bot/description/meshes/front_rgbd_camera_link.stl" scale="0.001 0.001 0.001"/>
-        </geometry>
+            <origin xyz="0 0 0.0225" rpy="0 0 0"/>
+            <geometry>
+                <box size="0.045 0.15 0.045"/>
+            </geometry>
         </collision>
     </link>
@@ -179,7 +179,7 @@
         </visual>
         <collision>
-            <origin xyz="0.6525 0 -0.705" rpy="0 0 1.5708"/>
-            <geometry>
-                <mesh filename="package://ros2-gz-vslam-bot/description/meshes/rear_rgbd_camera_link.stl" scale="0.001 0.001 0.001"/>
+            <origin xyz="0 0 0.0225" rpy="0 0 0"/>
+            <geometry>
+                <box size="0.045 0.15 0.045"/>
             </geometry>
         </collision>
@@ -202,7 +202,7 @@
         </visual>
         <collision>
-            <origin xyz="-0.58 0 -0.785" rpy="0 0 1.5708"/>
-            <geometry>
-                <mesh filename="package://ros2-gz-vslam-bot/description/meshes/front_livox_lidar_link.stl" scale="0.001 0.001 0.001"/>
+            <origin xyz="0 0 0.0375" rpy="0 0 0"/>
+            <geometry>
+                <cylinder radius="0.05" length="0.075"/>
             </geometry>
         </collision>
@@ -225,7 +225,7 @@
         </visual>
         <collision>
-            <origin xyz="0.58 0 -0.785" rpy="0 0 1.5708"/>
-            <geometry>
-                <mesh filename="package://ros2-gz-vslam-bot/description/meshes/rear_livox_lidar_link.stl" scale="0.001 0.001 0.001"/>
+            <origin xyz="0 0 0.0375" rpy="0 0 0"/>
+            <geometry>
+                <cylinder radius="0.05" length="0.075"/>
             </geometry>
         </collision>
