Commit message: fixing_bugs: #2

File: description/joints.xacro (robot description, xacro)
@@ -9,4 +9,5 @@
         <child link="l_f_wheel_link"/>
         <axis xyz="0.0 1.0 0.0"/>
+        <dynamics damping="1.0" friction="0.1"/>
     </joint>
     <joint name="l_r_wheel_joint" type="continuous">
@@ -15,4 +16,5 @@
         <child link="l_r_wheel_link"/>
         <axis xyz="0.0 1.0 0.0"/>
+        <dynamics damping="1.0" friction="0.1"/>
     </joint>
     <joint name="r_r_wheel_joint" type="continuous">
@@ -21,4 +23,5 @@
         <child link="r_r_wheel_link"/>
         <axis xyz="0.0 1.0 0.0"/>
+        <dynamics damping="1.0" friction="0.1"/>
     </joint>
     <joint name="r_f_wheel_joint" type="continuous">
@@ -27,4 +30,5 @@
         <child link="r_f_wheel_link"/>
         <axis xyz="0.0 1.0 0.0"/>
+        <dynamics damping="1.0" friction="0.1"/>
     </joint>
     <!-- =========================================== -->
