Commit message: edited the materials file

File: description/gazebo_materials.xacro (robot description, xacro)
@@ -2,26 +2,62 @@
 <robot xmlns:xacro="http://www.ros.org/wiki/xacro">
     <gazebo reference="base_link">
-        <material>Gazebo/White</material>
+        <material>
+            <ambient>0.820 0.710 0.550 1.000</ambient>
+            <diffuse>0.820 0.710 0.550 1.000</diffuse>
+        </material>
     </gazebo>
     <gazebo reference="l_f_wheel_link">
-        <material>Gazebo/Black</material>
+        <material>
+            <ambient>0 0 0 1</ambient>
+            <diffuse>0 0 0 1</diffuse>
+        </material>
     </gazebo>
     <gazebo reference="l_r_wheel_link">
-        <material>Gazebo/Black</material>
+        <material>
+            <ambient>0 0 0 1</ambient>
+            <diffuse>0 0 0 1</diffuse>
+        </material>
     </gazebo>
     <gazebo reference="r_f_wheel_link">
-        <material>Gazebo/Black</material>
+        <material>
+            <ambient>0 0 0 1</ambient>
+            <diffuse>0 0 0 1</diffuse>
+        </material>
     </gazebo>
     <gazebo reference="r_r_wheel_link">
-        <material>Gazebo/Black</material>
+        <material>
+            <ambient>0 0 0 1</ambient>
+            <diffuse>0 0 0 1</diffuse>
+        </material>
     </gazebo>
     <gazebo reference="front_bumper_link">
-        <material>Gazebo/Green</material>
+        <material>
+            <ambient>1 1 1 1</ambient>
+            <diffuse>1 1 1 1</diffuse>
+        </material>
     </gazebo>
     <gazebo reference="f_rgbd_link">
-        <material>Gazebo/Orange</material>
+        <material>
+            <ambient>0 1 0 1</ambient>
+            <diffuse>0 1 0 1</diffuse>
+        </material>
     </gazebo>
     <gazebo reference="r_rgbd_link">
-        <material>Gazebo/Orange</material>
+        <material>
+            <ambient>0 1 0 1</ambient>
+            <diffuse>0 1 0 1</diffuse>
+        </material>
+    </gazebo>
+    <gazebo reference="f_lidar_link">
+        <material>
+            <ambient>0 0 1 1</ambient>
+            <diffuse>0 0 1 1</diffuse>
+        </material>
+    </gazebo>
+    <gazebo reference="r_lidar_link">
+        <material>
+            <ambient>0 0 1 1</ambient>
+            <diffuse>0 0 1 1</diffuse>
+        </material>
     </gazebo>
 </robot>

Commit message: solving the wheel drift and wobbling issue

File: description/gazebo_materials.xacro (robot description, xacro)
@@ -7,4 +7,11 @@
         </material>
     </gazebo>
+    <!-- Anisotropic wheel friction: mu1 (fdir1 = rolling direction, local X)
+         kept high for straight-line traction; mu2 (lateral, local Y) lowered
+         so wheels can slide sideways during a skid-steer pivot without
+         stick-slip. kp/kd soften contact stiffness slightly to reduce
+         numerical jitter. Starting values — tune mu2 down further (e.g. 0.15)
+         if rocking persists, or up if the robot starts sliding out during
+         normal turns. -->
     <gazebo reference="l_f_wheel_link">
         <material>
@@ -12,4 +19,9 @@
             <diffuse>0 0 0 1</diffuse>
         </material>
+        <mu1>1.0</mu1>
+        <mu2>0.3</mu2>
+        <fdir1>1 0 0</fdir1>
+        <kp>1e6</kp>
+        <kd>10</kd>
     </gazebo>
     <gazebo reference="l_r_wheel_link">
@@ -18,4 +30,9 @@
             <diffuse>0 0 0 1</diffuse>
         </material>
+        <mu1>1.0</mu1>
+        <mu2>0.3</mu2>
+        <fdir1>1 0 0</fdir1>
+        <kp>1e6</kp>
+        <kd>10</kd>
     </gazebo>
     <gazebo reference="r_f_wheel_link">
@@ -24,4 +41,9 @@
             <diffuse>0 0 0 1</diffuse>
         </material>
+        <mu1>1.0</mu1>
+        <mu2>0.3</mu2>
+        <fdir1>1 0 0</fdir1>
+        <kp>1e6</kp>
+        <kd>10</kd>
     </gazebo>
     <gazebo reference="r_r_wheel_link">
@@ -30,6 +52,17 @@
             <diffuse>0 0 0 1</diffuse>
         </material>
+        <mu1>1.0</mu1>
+        <mu2>0.3</mu2>
+        <fdir1>1 0 0</fdir1>
+        <kp>1e6</kp>
+        <kd>10</kd>
     </gazebo>
     <gazebo reference="front_bumper_link">
+        <material>
+            <ambient>1 1 1 1</ambient>
+            <diffuse>1 1 1 1</diffuse>
+        </material>
+    </gazebo>
+    <gazebo reference="rear_bumper_link">
         <material>
             <ambient>1 1 1 1</ambient>

File: description/joints.xacro (robot description, xacro)
@@ -33,5 +33,5 @@
     </joint>
     <!-- =========================================== -->
-    <!-- ================ BUMPER JOINT ============= -->
+    <!-- ================ BUMPER JOINTS ============ -->
     <!-- =========================================== -->
     <joint name="front_bumper_joint" type="fixed">
@@ -39,4 +39,12 @@
         <parent link="base_link"/>
         <child link="front_bumper_link"/>
+    </joint>
+    <!-- Mirrors front_bumper_joint across the YZ plane (X negated) to
+         counterbalance the front bumper's mass and pull the whole-robot
+         center of mass back toward base_link's origin. -->
+    <joint name="rear_bumper_joint" type="fixed">
+        <origin xyz="-0.7 0.225 0.45" rpy="0 0 0"/>
+        <parent link="base_link"/>
+        <child link="rear_bumper_link"/>
     </joint>
     <!-- =========================================== -->

File: description/links.xacro (robot description, xacro)
@@ -140,4 +140,27 @@
     </link>
     <!-- =========================================== -->
+    <!-- ============= REAR BUMPER ================= -->
+    <!-- =========================================== -->
+    <link name="rear_bumper_link">
+        <inertial>
+            <origin xyz="-0.071440 -0.225000 -0.018717" rpy="0 0 0"/>
+            <mass value="13.822332678327909"/>
+            <inertia ixx="1.050773" iyy="0.249928" izz="0.823861" ixy="0.0" iyz="0.0" ixz="-0.000988"/>
+        </inertial>
+        <visual>
+            <origin xyz="0.7 -0.225 -0.45" rpy="0 0 -1.5708"/>
+            <geometry>
+                <mesh filename="package://ros2-gz-vslam-bot/description/meshes/front_bumper_link.stl" scale="0.001 0.001 0.001"/>
+            </geometry>
+            <material name="white"/>
+        </visual>
+        <collision>
+            <origin xyz="-0.071440 -0.225000 -0.018717" rpy="0 0 0"/>
+            <geometry>
+                <box size="0.12 0.95 0.5"/>
+            </geometry>
+        </collision>
+    </link>
+    <!-- =========================================== -->
     <!-- ========== FRONT RGBD CAMERA ============== -->
     <!-- =========================================== -->
