Commit message: edited the links file to support the repo name for meshes

File: description/links.xacro (robot description, xacro)
@@ -13,5 +13,5 @@
             <origin xyz="0 0 0" rpy="0 0 1.5708"/>
             <geometry>
-                <mesh filename="package://eos_v2/meshes/base_link.stl" scale="0.001 0.001 0.001"/>
+                <mesh filename="package://ros2-gz-vslam-bot/description/meshes/base_link.stl" scale="0.001 0.001 0.001"/>
             </geometry>
             <material name="desert_tan"/>
@@ -20,5 +20,5 @@
             <origin xyz="0 0 0" rpy="0 0 1.5708"/>
             <geometry>
-                <mesh filename="package://eos_v2/meshes/base_link.stl" scale="0.001 0.001 0.001"/>
+                <mesh filename="package://ros2-gz-vslam-bot/description/meshes/base_link.stl" scale="0.001 0.001 0.001"/>
             </geometry>
         </collision>
@@ -36,5 +36,5 @@
             <origin xyz="-0.45 -0.325 -0.225" rpy="0 0 1.5708"/>
             <geometry>
-                <mesh filename="package://eos_v2/meshes/left_front_wheel_link.stl" scale="0.001 0.001 0.001"/>
+                <mesh filename="package://ros2-gz-vslam-bot/description/meshes/left_front_wheel_link.stl" scale="0.001 0.001 0.001"/>
             </geometry>
             <material name="black"/>
@@ -43,5 +43,5 @@
             <origin xyz="-0.45 -0.325 -0.225" rpy="0 0 1.5708"/>
             <geometry>
-                <mesh filename="package://eos_v2/meshes/left_front_wheel_link.stl" scale="0.001 0.001 0.001"/>
+                <mesh filename="package://ros2-gz-vslam-bot/description/meshes/left_front_wheel_link.stl" scale="0.001 0.001 0.001"/>
             </geometry>
         </collision>
@@ -59,5 +59,5 @@
             <origin xyz="-0.45 0.325 -0.225" rpy="0 0 1.5708"/>
             <geometry>
-                <mesh filename="package://eos_v2/meshes/right_front_wheel_link.stl" scale="0.001 0.001 0.001"/>
+                <mesh filename="package://ros2-gz-vslam-bot/description/meshes/right_front_wheel_link.stl" scale="0.001 0.001 0.001"/>
             </geometry>
             <material name="black"/>
@@ -66,5 +66,5 @@
             <origin xyz="-0.45 0.325 -0.225" rpy="0 0 1.5708"/>
             <geometry>
-                <mesh filename="package://eos_v2/meshes/right_front_wheel_link.stl" scale="0.001 0.001 0.001"/>
+                <mesh filename="package://ros2-gz-vslam-bot/description/meshes/right_front_wheel_link.stl" scale="0.001 0.001 0.001"/>
             </geometry>
         </collision>
@@ -82,5 +82,5 @@
             <origin xyz="0.45 -0.325 -0.225" rpy="0 0 1.5708"/>
             <geometry>
-                <mesh filename="package://eos_v2/meshes/left_rear_wheel_link.stl" scale="0.001 0.001 0.001"/>
+                <mesh filename="package://ros2-gz-vslam-bot/description/meshes/left_rear_wheel_link.stl" scale="0.001 0.001 0.001"/>
             </geometry>
             <material name="black"/>
@@ -89,5 +89,5 @@
             <origin xyz="0.45 -0.325 -0.225" rpy="0 0 1.5708"/>
             <geometry>
-                <mesh filename="package://eos_v2/meshes/left_rear_wheel_link.stl" scale="0.001 0.001 0.001"/>
+                <mesh filename="package://ros2-gz-vslam-bot/description/meshes/left_rear_wheel_link.stl" scale="0.001 0.001 0.001"/>
             </geometry>
         </collision>
@@ -105,5 +105,5 @@
             <origin xyz="0.45 0.325 -0.225" rpy="0 0 1.5708"/>
             <geometry>
-                <mesh filename="package://eos_v2/meshes/right_rear_wheel_link.stl" scale="0.001 0.001 0.001"/>
+                <mesh filename="package://ros2-gz-vslam-bot/description/meshes/right_rear_wheel_link.stl" scale="0.001 0.001 0.001"/>
             </geometry>
             <material name="black"/>
@@ -112,5 +112,5 @@
             <origin xyz="0.45 0.325 -0.225" rpy="0 0 1.5708"/>
             <geometry>
-                <mesh filename="package://eos_v2/meshes/right_rear_wheel_link.stl" scale="0.001 0.001 0.001"/>
+                <mesh filename="package://ros2-gz-vslam-bot/description/meshes/right_rear_wheel_link.stl" scale="0.001 0.001 0.001"/>
             </geometry>
         </collision>
@@ -128,5 +128,5 @@
             <origin xyz="-0.7 -0.225 -0.45" rpy="0 0 1.5708"/>
             <geometry>
-                <mesh filename="package://eos_v2/meshes/front_bumper_link.stl" scale="0.001 0.001 0.001"/>
+                <mesh filename="package://ros2-gz-vslam-bot/description/meshes/front_bumper_link.stl" scale="0.001 0.001 0.001"/>
             </geometry>
             <material name="white"/>
@@ -135,5 +135,5 @@
             <origin xyz="-0.7 -0.225 -0.45" rpy="0 0 1.5708"/>
             <geometry>
-                <mesh filename="package://eos_v2/meshes/front_bumper_link.stl" scale="0.001 0.001 0.001"/>
+                <mesh filename="package://ros2-gz-vslam-bot/description/meshes/front_bumper_link.stl" scale="0.001 0.001 0.001"/>
             </geometry>
         </collision>
@@ -151,5 +151,5 @@
             <origin xyz="-0.6525 0 -0.705" rpy="0 0 1.5708"/>
             <geometry>
-            <mesh filename="package://eos_v2/meshes/front_rgbd_camera_link.stl" scale="0.001 0.001 0.001"/>
+            <mesh filename="package://ros2-gz-vslam-bot/description/meshes/front_rgbd_camera_link.stl" scale="0.001 0.001 0.001"/>
         </geometry>
             <material name="green"/>
@@ -158,5 +158,5 @@
             <origin xyz="-0.6525 0 -0.705" rpy="0 0 1.5708"/>
             <geometry>
-            <mesh filename="package://eos_v2/meshes/front_rgbd_camera_link.stl" scale="0.001 0.001 0.001"/>
+            <mesh filename="package://ros2-gz-vslam-bot/description/meshes/front_rgbd_camera_link.stl" scale="0.001 0.001 0.001"/>
         </geometry>
         </collision>
@@ -174,5 +174,5 @@
             <origin xyz="0.6525 0 -0.705" rpy="0 0 1.5708"/>
             <geometry>
-                <mesh filename="package://eos_v2/meshes/rear_rgbd_camera_link.stl" scale="0.001 0.001 0.001"/>
+                <mesh filename="package://ros2-gz-vslam-bot/description/meshes/rear_rgbd_camera_link.stl" scale="0.001 0.001 0.001"/>
             </geometry>
             <material name="green"/>
@@ -181,5 +181,5 @@
             <origin xyz="0.6525 0 -0.705" rpy="0 0 1.5708"/>
             <geometry>
-                <mesh filename="package://eos_v2/meshes/rear_rgbd_camera_link.stl" scale="0.001 0.001 0.001"/>
+                <mesh filename="package://ros2-gz-vslam-bot/description/meshes/rear_rgbd_camera_link.stl" scale="0.001 0.001 0.001"/>
             </geometry>
         </collision>
@@ -197,5 +197,5 @@
             <origin xyz="-0.58 0 -0.785" rpy="0 0 1.5708"/>
             <geometry>
-                <mesh filename="package://eos_v2/meshes/front_livox_lidar_link.stl" scale="0.001 0.001 0.001"/>
+                <mesh filename="package://ros2-gz-vslam-bot/description/meshes/front_livox_lidar_link.stl" scale="0.001 0.001 0.001"/>
             </geometry>
             <material name="blue"/>
@@ -204,5 +204,5 @@
             <origin xyz="-0.58 0 -0.785" rpy="0 0 1.5708"/>
             <geometry>
-                <mesh filename="package://eos_v2/meshes/front_livox_lidar_link.stl" scale="0.001 0.001 0.001"/>
+                <mesh filename="package://ros2-gz-vslam-bot/description/meshes/front_livox_lidar_link.stl" scale="0.001 0.001 0.001"/>
             </geometry>
         </collision>
@@ -220,5 +220,5 @@
             <origin xyz="0.58 0 -0.785" rpy="0 0 1.5708"/>
             <geometry>
-                <mesh filename="package://eos_v2/meshes/rear_livox_lidar_link.stl" scale="0.001 0.001 0.001"/>
+                <mesh filename="package://ros2-gz-vslam-bot/description/meshes/rear_livox_lidar_link.stl" scale="0.001 0.001 0.001"/>
             </geometry>
             <material name="blue"/>
@@ -227,5 +227,5 @@
             <origin xyz="0.58 0 -0.785" rpy="0 0 1.5708"/>
             <geometry>
-                <mesh filename="package://eos_v2/meshes/rear_livox_lidar_link.stl" scale="0.001 0.001 0.001"/>
+                <mesh filename="package://ros2-gz-vslam-bot/description/meshes/rear_livox_lidar_link.stl" scale="0.001 0.001 0.001"/>
             </geometry>
         </collision>

Commit message: changed wheel collision from cylinder to sphere for testing

File: description/links.xacro (robot description, xacro)
@@ -43,5 +43,5 @@
             <origin xyz="0 0.11207 0" rpy="1.5708 0 0"/>
             <geometry>
-                <cylinder radius="0.225" length="0.125"/>
+                <sphere radius="0.225"/>
             </geometry>
         </collision>
@@ -66,5 +66,5 @@
             <origin xyz="0 -0.11207 0" rpy="1.5708 0 0"/>
             <geometry>
-                <cylinder radius="0.225" length="0.125"/>
+                <sphere radius="0.225"/>
             </geometry>
         </collision>
@@ -89,5 +89,5 @@
             <origin xyz="0 0.11207 0" rpy="1.5708 0 0"/>
             <geometry>
-                <cylinder radius="0.225" length="0.125"/>
+                <sphere radius="0.225"/>
             </geometry>
         </collision>
@@ -112,5 +112,5 @@
             <origin xyz="0 -0.11207 0" rpy="1.5708 0 0"/>
             <geometry>
-                <cylinder radius="0.225" length="0.125"/>
+                <sphere radius="0.225"/>
             </geometry>
         </collision>
