Commit message: edited the links and sensors file ot add lidars file

File: description/gazebo_sensors.xacro (robot description, xacro)
@@ -5,6 +5,9 @@
     <!-- =========================================== -->
     <gazebo reference="f_rgbd_link">
-        <sensor name="front camera" type="depth">
+        <sensor name="front_camera" type="rgbd_camera">
             <update_rate>20</update_rate>
+            <always_on>1</always_on>
+            <visualize>true</visualize>
+            <topic>camera/front</topic>
             <camera>
                 <horizontal_fov>1.089</horizontal_fov>
@@ -19,9 +22,4 @@
                 </clip>
             </camera>
-            <plugin name="camera_controller" filename="libgazebo_ros_camera.so">
-                <frame_name>camera_optical_frame</frame_name>
-                <min_depth>0.1</min_depth>
-                <max_depth>8.0</max_depth>
-            </plugin>
         </sensor>
     </gazebo>
@@ -30,6 +28,9 @@
     <!-- =========================================== -->
     <gazebo reference="r_rgbd_link">
-        <sensor name="rear camera" type="depth">
+        <sensor name="rear_camera" type="rgbd_camera">
             <update_rate>20</update_rate>
+            <always_on>1</always_on>
+            <visualize>true</visualize>
+            <topic>camera/rear</topic>
             <camera>
                 <horizontal_fov>1.089</horizontal_fov>
@@ -44,9 +45,68 @@
                 </clip>
             </camera>
-            <plugin name="camera_controller" filename="libgazebo_ros_camera.so">
-                <frame_name>camera_optical_frame</frame_name>
-                <min_depth>0.1</min_depth>
-                <max_depth>8.0</max_depth>
-            </plugin>
+        </sensor>
+    </gazebo>
+    <!-- =========================================== -->
+    <!-- ========== FRONT LIDAR SENSOR ============= -->
+    <!-- =========================================== -->
+    <gazebo reference="f_lidar_link">
+        <sensor name="front_lidar" type="gpu_lidar">
+            <update_rate>10</update_rate>
+            <always_on>1</always_on>
+            <visualize>true</visualize>
+            <topic>lidar/front/scan</topic>
+            <lidar>
+                <scan>
+                    <horizontal>
+                        <samples>640</samples>
+                        <resolution>1</resolution>
+                        <min_angle>-3.14159</min_angle>
+                        <max_angle>3.14159</max_angle>
+                    </horizontal>
+                    <vertical>
+                        <samples>16</samples>
+                        <resolution>1</resolution>
+                        <min_angle>-0.2618</min_angle>
+                        <max_angle>0.2618</max_angle>
+                    </vertical>
+                </scan>
+                <range>
+                    <min>0.1</min>
+                    <max>30.0</max>
+                    <resolution>0.01</resolution>
+                </range>
+            </lidar>
+        </sensor>
+    </gazebo>
+    <!-- =========================================== -->
+    <!-- ========== REAR LIDAR SENSOR =============== -->
+    <!-- =========================================== -->
+    <gazebo reference="r_lidar_link">
+        <sensor name="rear_lidar" type="gpu_lidar">
+            <update_rate>10</update_rate>
+            <always_on>1</always_on>
+            <visualize>true</visualize>
+            <topic>lidar/rear/scan</topic>
+            <lidar>
+                <scan>
+                    <horizontal>
+                        <samples>640</samples>
+                        <resolution>1</resolution>
+                        <min_angle>-3.14159</min_angle>
+                        <max_angle>3.14159</max_angle>
+                    </horizontal>
+                    <vertical>
+                        <samples>16</samples>
+                        <resolution>1</resolution>
+                        <min_angle>-0.2618</min_angle>
+                        <max_angle>0.2618</max_angle>
+                    </vertical>
+                </scan>
+                <range>
+                    <min>0.1</min>
+                    <max>30.0</max>
+                    <resolution>0.01</resolution>
+                </range>
+            </lidar>
         </sensor>
     </gazebo>

File: description/links.xacro (robot description, xacro)
@@ -185,3 +185,49 @@
         </collision>
   </link>
+    <!-- =========================================== -->
+    <!-- ========== FRONT LIVOX LIDAR ============== -->
+    <!-- =========================================== -->
+    <link name="f_lidar_link">
+        <inertial>
+            <origin xyz="0 0 0.0375" rpy="0 0 0"/>
+            <mass value="1.0750137361502572"/>
+            <inertia ixx="0.001176" iyy="0.001176" izz="0.001344" ixy="0.0" iyz="0.0" ixz="0.0"/>
+        </inertial>
+        <visual>
+            <origin xyz="-0.58 0 -0.785" rpy="0 0 1.5708"/>
+            <geometry>
+                <mesh filename="package://eos_v2/meshes/front_livox_lidar_link.stl" scale="0.001 0.001 0.001"/>
+            </geometry>
+            <material name="blue"/>
+        </visual>
+        <collision>
+            <origin xyz="-0.58 0 -0.785" rpy="0 0 1.5708"/>
+            <geometry>
+                <mesh filename="package://eos_v2/meshes/front_livox_lidar_link.stl" scale="0.001 0.001 0.001"/>
+            </geometry>
+        </collision>
+    </link>
+    <!-- =========================================== -->
+    <!-- =========== REAR LIVOX LIDAR =============== -->
+    <!-- =========================================== -->
+    <link name="r_lidar_link">
+        <inertial>
+            <origin xyz="0 0 0.0375" rpy="0 0 0"/>
+            <mass value="1.0750137361502572"/>
+            <inertia ixx="0.001176" iyy="0.001176" izz="0.001344" ixy="0.0" iyz="0.0" ixz="0.0"/>
+        </inertial>
+        <visual>
+            <origin xyz="0.58 0 -0.785" rpy="0 0 1.5708"/>
+            <geometry>
+                <mesh filename="package://eos_v2/meshes/rear_livox_lidar_link.stl" scale="0.001 0.001 0.001"/>
+            </geometry>
+            <material name="blue"/>
+        </visual>
+        <collision>
+            <origin xyz="0.58 0 -0.785" rpy="0 0 1.5708"/>
+            <geometry>
+                <mesh filename="package://eos_v2/meshes/rear_livox_lidar_link.stl" scale="0.001 0.001 0.001"/>
+            </geometry>
+        </collision>
+    </link>
 </robot>

Commit message: separated camera into two different sensors, working on fixing depth side

File: description/gazebo_sensors.xacro (robot description, xacro)
@@ -2,15 +2,21 @@
 <robot xmlns:xacro="http://www.ros.org/wiki/xacro">
     <!-- =========================================== -->
-    <!-- ========== FRONT CAMERA SENSOR ============ -->
+    <!-- ========== FRONT CAMERA SENSORS ============ -->
     <!-- =========================================== -->
+    <!-- Split into two separate sensors instead of one combined rgbd_camera.
+         This exercises different gz-sensors code (CameraSensor / DepthCameraSensor)
+         than the combined RgbdCameraSensor implementation, which showed
+         intermittent frame corruption on ogre2 during robot motion
+         (matches gazebosim/ros_gz#738, closed upstream with no fix).
+         Trade-off: no fused colored point cloud output anymore — if your
+         VSLAM framework needs that, this will need revisiting. Frameworks
+         that sync separate RGB + depth + camera_info topics (e.g. RTAB-Map)
+         are unaffected. -->
     <gazebo reference="f_rgbd_link">
-        <sensor name="front_camera" type="rgbd_camera">
-            <pose>0 0 0 0 0 0</pose>
+        <sensor name="front_camera" type="camera">
             <update_rate>30</update_rate>
             <visualize>true</visualize>
-            <always_on>true</always_on>
-            <topic>camera/front</topic>
-            <gz_frame_id>f_rgbd_link</gz_frame_id>
-            <camera name="front_camera">
+            <topic>camera/front/image</topic>
+            <camera>
                 <horizontal_fov>1.089</horizontal_fov>
                 <image>
@@ -23,16 +29,36 @@
                     <far>20.0</far>
                 </clip>
+                <camera_info_topic>camera/front/camera_info</camera_info_topic>
+            </camera>
+        </sensor>
+    </gazebo>
+    <gazebo reference="f_rgbd_link">
+        <sensor name="front_depth_camera" type="depth_camera">
+            <update_rate>30</update_rate>
+            <visualize>true</visualize>
+            <topic>camera/front/depth_image</topic>
+            <camera>
+                <horizontal_fov>1.089</horizontal_fov>
+                <image>
+                    <width>640</width>
+                    <height>480</height>
+                    <format>R_FLOAT32</format>
+                </image>
+                <clip>
+                    <near>0.05</near>
+                    <far>20.0</far>
+                </clip>
             </camera>
         </sensor>
     </gazebo>
     <!-- =========================================== -->
-    <!-- =========== REAR CAMERA SENSOR ============ -->
+    <!-- =========== REAR CAMERA SENSORS ============ -->
     <!-- =========================================== -->
     <gazebo reference="r_rgbd_link">
-        <sensor name="rear_camera" type="rgbd_camera">
+        <sensor name="rear_camera" type="camera">
             <update_rate>20</update_rate>
             <always_on>1</always_on>
             <visualize>true</visualize>
-            <topic>camera/rear</topic>
+            <topic>camera/rear/image</topic>
             <camera>
                 <horizontal_fov>1.089</horizontal_fov>
@@ -41,4 +67,25 @@
                     <height>480</height>
                     <format>R8G8B8</format>
+                </image>
+                <clip>
+                    <near>0.05</near>
+                    <far>20.0</far>
+                </clip>
+                <camera_info_topic>camera/rear/camera_info</camera_info_topic>
+            </camera>
+        </sensor>
+    </gazebo>
+    <gazebo reference="r_rgbd_link">
+        <sensor name="rear_depth_camera" type="depth_camera">
+            <update_rate>20</update_rate>
+            <always_on>1</always_on>
+            <visualize>true</visualize>
+            <topic>camera/rear/depth_image</topic>
+            <camera>
+                <horizontal_fov>1.089</horizontal_fov>
+                <image>
+                    <width>640</width>
+                    <height>480</height>
+                    <format>R_FLOAT32</format>
                 </image>
                 <clip>

File: description/links.xacro (robot description, xacro)
@@ -11,7 +11,8 @@
     	</inertial>
     	<visual>
+    	    <origin xyz="0.000973 0.000007 0.486096" rpy="0 0 0"/>
             <origin xyz="0 0 0" rpy="0 0 1.5708"/>
             <geometry>
-                <mesh filename="package://ros2-gz-vslam-bot/description/meshes/base_link.stl" scale="0.001 0.001 0.001"/>
+                <box size="1.35 0.75 0.30"/>
             </geometry>
             <material name="desert_tan"/>
@@ -34,7 +35,7 @@
         </inertial>
         <visual>
-            <origin xyz="-0.45 -0.325 -0.225" rpy="0 0 1.5708"/>
-            <geometry>
-                <mesh filename="package://ros2-gz-vslam-bot/description/meshes/left_front_wheel_link.stl" scale="0.001 0.001 0.001"/>
+            <origin xyz="0 0.11207 0" rpy="1.5708 0 0"/>
+            <geometry>
+                <cylinder radius="0.225" length="0.125"/>
             </geometry>
             <material name="black"/>
@@ -57,7 +58,7 @@
         </inertial>
         <visual>
-            <origin xyz="-0.45 0.325 -0.225" rpy="0 0 1.5708"/>
-            <geometry>
-                <mesh filename="package://ros2-gz-vslam-bot/description/meshes/right_front_wheel_link.stl" scale="0.001 0.001 0.001"/>
+            <origin xyz="0 -0.11207 0" rpy="1.5708 0 0"/>
+            <geometry>
+                <cylinder radius="0.225" length="0.125"/>
             </geometry>
             <material name="black"/>
@@ -80,7 +81,7 @@
         </inertial>
         <visual>
-            <origin xyz="0.45 -0.325 -0.225" rpy="0 0 1.5708"/>
-            <geometry>
-                <mesh filename="package://ros2-gz-vslam-bot/description/meshes/left_rear_wheel_link.stl" scale="0.001 0.001 0.001"/>
+            <origin xyz="0 0.11207 0" rpy="1.5708 0 0"/>
+            <geometry>
+                <cylinder radius="0.225" length="0.125"/>
             </geometry>
             <material name="black"/>
@@ -103,7 +104,7 @@
         </inertial>
         <visual>
-            <origin xyz="0.45 0.325 -0.225" rpy="0 0 1.5708"/>
-            <geometry>
-                <mesh filename="package://ros2-gz-vslam-bot/description/meshes/right_rear_wheel_link.stl" scale="0.001 0.001 0.001"/>
+            <origin xyz="0 -0.11207 0" rpy="1.5708 0 0"/>
+            <geometry>
+                <cylinder radius="0.225" length="0.125"/>
             </geometry>
             <material name="black"/>
@@ -126,7 +127,7 @@
         </inertial>
         <visual>
-            <origin xyz="-0.7 -0.225 -0.45" rpy="0 0 1.5708"/>
-            <geometry>
-                <mesh filename="package://ros2-gz-vslam-bot/description/meshes/front_bumper_link.stl" scale="0.001 0.001 0.001"/>
+            <origin xyz="0.071440 -0.225000 -0.018717" rpy="0 0 0"/>
+            <geometry>
+                <box size="0.12 0.95 0.4"/>
             </geometry>
             <material name="white"/>
@@ -135,5 +136,5 @@
             <origin xyz="0.071440 -0.225000 -0.018717" rpy="0 0 0"/>
             <geometry>
-                <box size="0.12 0.95 0.5"/>
+                <box size="0.12 0.95 0.4"/>
             </geometry>
         </collision>
@@ -149,7 +150,7 @@
         </inertial>
         <visual>
-            <origin xyz="0.7 -0.225 -0.45" rpy="0 0 -1.5708"/>
-            <geometry>
-                <mesh filename="package://ros2-gz-vslam-bot/description/meshes/front_bumper_link.stl" scale="0.001 0.001 0.001"/>
+            <origin xyz="-0.071440 -0.225000 -0.018717" rpy="0 0 0"/>
+            <geometry>
+                <box size="0.12 0.95 0.4"/>
             </geometry>
             <material name="white"/>
@@ -158,5 +159,5 @@
             <origin xyz="-0.071440 -0.225000 -0.018717" rpy="0 0 0"/>
             <geometry>
-                <box size="0.12 0.95 0.5"/>
+                <box size="0.12 0.95 0.4"/>
             </geometry>
         </collision>
@@ -218,7 +219,7 @@
         </inertial>
         <visual>
-            <origin xyz="-0.58 0 -0.785" rpy="0 0 1.5708"/>
-            <geometry>
-                <mesh filename="package://ros2-gz-vslam-bot/description/meshes/front_livox_lidar_link.stl" scale="0.001 0.001 0.001"/>
+            <origin xyz="0 0 0.0375" rpy="0 0 0"/>
+            <geometry>
+                <cylinder radius="0.05" length="0.075"/>
             </geometry>
             <material name="blue"/>
@@ -241,7 +242,7 @@
         </inertial>
         <visual>
-            <origin xyz="0.58 0 -0.785" rpy="0 0 1.5708"/>
-            <geometry>
-                <mesh filename="package://ros2-gz-vslam-bot/description/meshes/rear_livox_lidar_link.stl" scale="0.001 0.001 0.001"/>
+            <origin xyz="0 0 0.0375" rpy="0 0 0"/>
+            <geometry>
+                <cylinder radius="0.05" length="0.075"/>
             </geometry>
             <material name="blue"/>
