Commit message: removed meshes for easier compute and made the visuals a bit better

File: description/gazebo_sensors.xacro (robot description, xacro)
@@ -27,5 +27,5 @@
                 <clip>
                     <near>0.05</near>
-                    <far>400.0</far>
+                    <far>20.0</far>
                 </clip>
                 <camera_info_topic>camera/front/camera_info</camera_info_topic>
@@ -53,12 +53,24 @@
     </gazebo>
     <!-- =========================================== -->
-    <!-- =========== REAR CAMERA SENSORS ============ -->
+    <!-- =========== REAR CAMERA SENSOR ============ -->
     <!-- =========================================== -->
+    <!-- Combined rgbd_camera sensor, per request, modeled on a found
+         reference example (visualize=false, nested depth_camera clip
+         range adopted; noise/distortion/custom intrinsics/L8 format and
+         $(arg ns) syntax deliberately NOT carried over).
+         NOTE: this is the same sensor type that caused front camera's
+         motion-triggered corruption bug (matches gazebosim/ros_gz#738)
+         before front was split into separate camera + depth_camera
+         sensors. Rear was never independently tested for this bug —
+         this is an accepted risk. If rear shows the same flat/corrupted
+         frames during motion, the fix that worked for front (splitting
+         into separate camera + depth_camera sensors, see f_rgbd_link's
+         blocks above) will work here too. -->
     <gazebo reference="r_rgbd_link">
-        <sensor name="rear_camera" type="camera">
+        <sensor name="rear_camera" type="rgbd_camera">
             <update_rate>20</update_rate>
             <always_on>1</always_on>
-            <visualize>true</visualize>
-            <topic>camera/rear/image</topic>
+            <visualize>false</visualize>
+            <topic>camera/rear</topic>
             <camera>
                 <horizontal_fov>1.089</horizontal_fov>
@@ -70,27 +82,17 @@
                 <clip>
                     <near>0.05</near>
-                    <far>400.0</far>
-                </clip>
-                <camera_info_topic>camera/rear/camera_info</camera_info_topic>
-            </camera>
-        </sensor>
-    </gazebo>
-    <gazebo reference="r_rgbd_link">
-        <sensor name="rear_depth_camera" type="depth_camera">
-            <update_rate>20</update_rate>
-            <always_on>1</always_on>
-            <visualize>true</visualize>
-            <topic>camera/rear/depth_image</topic>
-            <camera>
-                <horizontal_fov>1.089</horizontal_fov>
-                <image>
-                    <width>640</width>
-                    <height>480</height>
-                    <format>R_FLOAT32</format>
-                </image>
-                <clip>
-                    <near>0.05</near>
                     <far>20.0</far>
                 </clip>
+                <!-- Separate, tighter clip range specifically for the depth
+                     output, adopted from the reference example — typical
+                     of real RGBD hardware (depth range is usually shorter
+                     than the color image's usable range). Adjust if you
+                     want depth to match the full 20m color range instead. -->
+                <depth_camera>
+                    <clip>
+                        <near>0.1</near>
+                        <far>10.0</far>
+                    </clip>
+                </depth_camera>
             </camera>
         </sensor>

File: description/joints.xacro (robot description, xacro)
@@ -52,10 +52,10 @@
     <!-- =========================================== -->
     <joint name="f_rgbd_joint" type="fixed">
-        <origin xyz="0.6525 0.0 0.705" rpy="0 0 0"/>
+        <origin xyz="0.6525 0.0 0.6625" rpy="0 0 0"/>
         <parent link="base_link"/>
         <child link="f_rgbd_link"/>
     </joint>
     <joint name="r_rgbd_joint" type="fixed">
-        <origin xyz="-0.6525 0.0 0.705" rpy="0 0 0"/>
+        <origin xyz="-0.6525 0.0 0.6625" rpy="0 0 ${pi}"/>
         <parent link="base_link"/>
         <child link="r_rgbd_link"/>
@@ -65,10 +65,10 @@
     <!-- =========================================== -->
     <joint name="f_lidar_joint" type="fixed">
-        <origin xyz="0.58 0.0 0.785" rpy="0 0 0"/>
+        <origin xyz="0.55 0.0 0.74" rpy="0 0 0"/>
         <parent link="base_link"/>
         <child link="f_lidar_link"/>
     </joint>
     <joint name="r_lidar_joint" type="fixed">
-        <origin xyz="-0.58 0.0 0.785" rpy="0 0 0"/>
+        <origin xyz="-0.55 0.0 0.74" rpy="0 0 ${pi}"/>
         <parent link="base_link"/>
         <child link="r_lidar_link"/>

File: description/links.xacro (robot description, xacro)
@@ -12,7 +12,20 @@
     	<visual>
     	    <origin xyz="0.000973 0.000007 0.486096" rpy="0 0 0"/>
-            <origin xyz="0 0 0" rpy="0 0 1.5708"/>
             <geometry>
                 <box size="1.35 0.75 0.30"/>
+            </geometry>
+            <material name="desert_tan"/>
+        </visual>
+        <visual>
+    	    <origin xyz="0.55 0.0 0.685" rpy="0 0 0"/>
+            <geometry>
+                <cylinder radius="0.05" length="0.1"/>
+            </geometry>
+            <material name="desert_tan"/>
+        </visual>
+         <visual>
+    	    <origin xyz="-0.55 0.0 0.685" rpy="0 0 0"/>
+            <geometry>
+                <cylinder radius="0.05" length="0.1"/>
             </geometry>
             <material name="desert_tan"/>
@@ -173,14 +186,25 @@
         </inertial>
         <visual>
-            <origin xyz="-0.6525 0 -0.705" rpy="0 0 1.5708"/>
-            <geometry>
-            <mesh filename="package://ros2-gz-vslam-bot/description/meshes/front_rgbd_camera_link.stl" scale="0.001 0.001 0.001"/>
-        </geometry>
-            <material name="green"/>
-        </visual>
-        <collision>
-            <origin xyz="0 0 0.0225" rpy="0 0 0"/>
-            <geometry>
-                <box size="0.045 0.15 0.045"/>
+            <geometry>
+                <box size="0.05 0.05 0.05"/>
+            </geometry>
+            <material name="green"/>
+        </visual>
+        <visual>
+            <origin xyz="0.035 0 0" rpy="0 ${pi/2} 0"/>
+            <geometry>
+                <cylinder radius="0.015" length="0.02"/>
+            </geometry>
+            <material name="green"/>
+        </visual>
+        <collision>
+            <geometry>
+                <box size="0.05 0.05 0.05"/>
+            </geometry>
+        </collision>
+        <collision>
+            <origin xyz="0.035 0 0" rpy="0 ${pi/2} 0"/>
+            <geometry>
+                <cylinder radius="0.015" length="0.02"/>
             </geometry>
         </collision>
@@ -196,14 +220,25 @@
         </inertial>
         <visual>
-            <origin xyz="0.6525 0 -0.705" rpy="0 0 1.5708"/>
-            <geometry>
-                <mesh filename="package://ros2-gz-vslam-bot/description/meshes/rear_rgbd_camera_link.stl" scale="0.001 0.001 0.001"/>
-            </geometry>
-            <material name="green"/>
-        </visual>
-        <collision>
-            <origin xyz="0 0 0.0225" rpy="0 0 0"/>
-            <geometry>
-                <box size="0.045 0.15 0.045"/>
+            <geometry>
+                <box size="0.05 0.05 0.05"/>
+            </geometry>
+            <material name="green"/>
+        </visual>
+        <visual>
+            <origin xyz="0.035 0 0" rpy="0 ${pi/2} 0"/>
+            <geometry>
+                <cylinder radius="0.015" length="0.02"/>
+            </geometry>
+            <material name="green"/>
+        </visual>
+        <collision>
+            <geometry>
+                <box size="0.05 0.05 0.05"/>
+            </geometry>
+        </collision>
+        <collision>
+            <origin xyz="0.035 0 0" rpy="0 ${pi/2} 0"/>
+            <geometry>
+                <cylinder radius="0.015" length="0.02"/>
             </geometry>
         </collision>

Commit message: basic robot finally fixed

File: description/gazebo_sensors.xacro (robot description, xacro)
@@ -10,5 +10,5 @@
             <visualize>true</visualize>
             <update_rate>20</update_rate>
-            <topic>camera</topic>
+            <topic>camera/front</topic>
             <gz_frame_id>f_rgbd_link</gz_frame_id>
             <camera name="rgbd_camera">
@@ -23,5 +23,5 @@
                     <far>20.0</far>
                 </clip>
-                <camera_info_topic>camera/camera_info</camera_info_topic>
+                <camera_info_topic>camera/front/camera_info</camera_info_topic>
                 <depth_camera>
                     <clip>
@@ -42,5 +42,5 @@
             <visualize>true</visualize>
             <update_rate>20</update_rate>
-            <topic>camera2</topic>
+            <topic>camera/rear</topic>
             <gz_frame_id>r_rgbd_link</gz_frame_id>
             <camera name="rgbd_camera">
@@ -55,5 +55,5 @@
                     <far>20.0</far>
                 </clip>
-                <camera_info_topic>camera2/camera_info</camera_info_topic>
+                <camera_info_topic>camera/rear/camera_info</camera_info_topic>
                 <depth_camera>
                     <clip>

File: description/links.xacro (robot description, xacro)
@@ -142,5 +142,5 @@
             <origin xyz="0.071440 -0.225000 -0.018717" rpy="0 0 0"/>
             <geometry>
-                <box size="0.12 0.95 0.4"/>
+                <box size="0.12 0.95 0.3"/>
             </geometry>
             <material name="white"/>
@@ -149,5 +149,5 @@
             <origin xyz="0.071440 -0.225000 -0.018717" rpy="0 0 0"/>
             <geometry>
-                <box size="0.12 0.95 0.4"/>
+                <box size="0.12 0.95 0.3"/>
             </geometry>
         </collision>
@@ -165,5 +165,5 @@
             <origin xyz="-0.071440 -0.225000 -0.018717" rpy="0 0 0"/>
             <geometry>
-                <box size="0.12 0.95 0.4"/>
+                <box size="0.12 0.95 0.3"/>
             </geometry>
             <material name="white"/>
@@ -172,5 +172,5 @@
             <origin xyz="-0.071440 -0.225000 -0.018717" rpy="0 0 0"/>
             <geometry>
-                <box size="0.12 0.95 0.4"/>
+                <box size="0.12 0.95 0.3"/>
             </geometry>
         </collision>
